File: Schematic/MCU_MR/MCU_MR.kicad_sch (KiCad schematic)
At the start: 26 parts, among them J1 USB to TTL CP2102, J2 Power supply terminal, J3 PICKIT3, SW1 SW_Push, SW2 SW_Push, SW3 SW_Push, SW4 SW_Push, U1 PIC16F887-IP, Y1 20MHz

Commit message: Schematic: Update Kicad schematic
Parts:
- added C10: 100nF, symbol Device:C
- added C9: 470uF, symbol Device:C_Polarized
Connections:
- net +5V: now also C10.1, C9.1
- net GND: now also C10.2, C9.2

Commit message: Update THUYETMINH
Parts:
- C3, C4: value 100nF -> 22pF
Other:
- moved on the sheet: C10, C9, D9, R10
Changed lines of the file:
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@@
 	)
 	(junction
-		(at 77.47 21.59)
+		(at 87.63 22.86)
 		(diameter 0)
 		(color 0 0 0 0)
 	)
 	(junction
-		(at 88.9 21.59)
+		(at 99.06 22.86)
 		(diameter 0)
 		(color 0 0 0 0)
@@
 	)
 	(junction
-		(at 77.47 40.64)
+		(at 87.63 41.91)
 		(diameter 0)
 		(color 0 0 0 0)
@@
 	)
 	(junction
-		(at 88.9 40.64)
+		(at 99.06 41.91)
 		(diameter 0)
 		(color 0 0 0 0)
@@
 	(wire
 		(pts
-			(xy 88.9 21.59) (xy 88.9 25.4)
+			(xy 99.06 22.86) (xy 99.06 26.67)
 		)
 		(stroke
@@
 	(wire
 		(pts
-			(xy 88.9 21.59) (xy 101.6 21.59)
+			(xy 99.06 22.86) (xy 111.76 22.86)
 		)
 		(stroke
@@
 	(wire
 		(pts
-			(xy 77.47 21.59) (xy 77.47 22.86)
+			(xy 87.63 22.86) (xy 87.63 24.13)
 		)
 		(stroke
@@
 	(wire
 		(pts
-			(xy 77.47 40.64) (xy 88.9 40.64)
+			(xy 87.63 41.91) (xy 99.06 41.91)
 		)
 		(stroke
@@
 	(wire
 		(pts
-			(xy 77.47 30.48) (xy 77.47 31.75)
+			(xy 87.63 31.75) (xy 87.63 33.02)
 		)
 		(stroke
@@
 	(wire
 		(pts
-			(xy 88.9 33.02) (xy 88.9 40.64)
+			(xy 99.06 34.29) (xy 99.06 41.91)
 		)
 		(stroke
@@
 	(wire
 		(pts
-			(xy 77.47 21.59) (xy 88.9 21.59)
+			(xy 87.63 22.86) (xy 99.06 22.86)
 		)
 		(stroke
@@
 	(wire
 		(pts
-			(xy 77.47 40.64) (xy 77.47 41.91)
+			(xy 87.63 41.91) (xy 87.63 43.18)
 		)
 		(stroke
@@
 	(wire
 		(pts
-			(xy 101.6 21.59) (xy 101.6 25.4)
+			(xy 111.76 22.86) (xy 111.76 26.67)
 		)
 		(stroke
@@
 	(wire
 		(pts
-			(xy 77.47 20.32) (xy 77.47 21.59)
+			(xy 87.63 21.59) (xy 87.63 22.86)
 		)
 		(stroke
@@
 	(wire
 		(pts
-			(xy 77.47 39.37) (xy 77.47 40.64)
+			(xy 87.63 40.64) (xy 87.63 41.91)
 		)
 		(stroke
@@
 	(wire
 		(pts
-			(xy 101.6 40.64) (xy 101.6 33.02)
+			(xy 111.76 41.91) (xy 111.76 34.29)
 		)
 		(stroke
@@
 	(wire
 		(pts
-			(xy 88.9 40.64) (xy 101.6 40.64)
+			(xy 99.06 41.91) (xy 111.76 41.91)
 		)
 		(stroke
@@
 			)
 		)
-		(property "Value" "100nF"
+		(property "Value" "22pF"
 			(at 33.02 76.1999 0)
 			(effects
@@
 			)
 		)
-		(property "Value" "100nF"
+		(property "Value" "22pF"
 			(at 48.26 76.1999 0)
 			(effects
@@
 	(symbol
 		(lib_id "power:GND")
-		(at 77.47 41.91 0)
+		(at 87.63 43.18 0)
 		(unit 1)
 		(exclude_from_sim no)
@@
 		(fields_autoplaced yes)
 		(property "Reference" "#PWR021"
-			(at 77.47 48.26 0)
+			(at 87.63 49.53 0)
 			(effects
 				(font
@@
 		)
 		(property "Value" "GND"
-			(at 77.47 46.99 0)
+			(at 87.63 48.26 0)
 			(effects
 				(font
@@
 		)
 		(property "Footprint" ""
-			(at 77.47 41.91 0)
+			(at 87.63 43.18 0)
 			(effects
 				(font
@@
 		)
 		(property "Datasheet" ""
-			(at 77.47 41.91 0)
+			(at 87.63 43.18 0)
 			(effects
 				(font
@@
 		)
 		(property "Description" "Power symbol creates a global label with name \"GND\" , ground"
-			(at 77.47 41.91 0)
+			(at 87.63 43.18 0)
 			(effects
 				(font
@@
 	(symbol
 		(lib_id "power:+5V")
-		(at 77.47 20.32 0)
+		(at 87.63 21.59 0)
 		(unit 1)
 		(exclude_from_sim no)
@@
 		(fields_autoplaced yes)
 		(property "Reference" "#PWR020"
-			(at 77.47 24.13 0)
+			(at 87.63 25.4 0)
 			(effects
 				(font
@@
 		)
 		(property "Value" "+5V"
-			(at 77.47 15.24 0)
+			(at 87.63 16.51 0)
 			(effects
 				(font
@@
 		)
 		(property "Footprint" ""
-			(at 77.47 20.32 0)
+			(at 87.63 21.59 0)
 			(effects
 				(font
@@
 		)
 		(property "Datasheet" ""
-			(at 77.47 20.32 0)
+			(at 87.63 21.59 0)
 			(effects
 				(font
@@
 		)
 		(property "Description" "Power symbol creates a global label with name \"+5V\""
-			(at 77.47 20.32 0)
+			(at 87.63 21.59 0)
 			(effects
 				(font
@@
 	(symbol
 		(lib_id "Device:LED")
-		(at 77.47 35.56 90)
+		(at 87.63 36.83 90)
 		(unit 1)
 		(exclude_from_sim no)
@@
 		(fields_autoplaced yes)
 		(property "Reference" "D9"
-			(at 81.28 35.8774 90)
+			(at 91.44 37.1474 90)
 			(effects
 				(font
@@
 		)
 		(property "Value" "LED"
-			(at 81.28 38.4174 90)
+			(at 91.44 39.6874 90)
 			(effects
 				(font
@@
 		)
 		(property "Footprint" ""
-			(at 77.47 35.56 0)
+			(at 87.63 36.83 0)
 			(effects
 				(font
@@
 		)
 		(property "Datasheet" "~"
-			(at 77.47 35.56 0)
+			(at 87.63 36.83 0)
 			(effects
 				(font
@@
 		)
 		(property "Description" "Light emitting diode"
-			(at 77.47 35.56 0)
+			(at 87.63 36.83 0)
 			(effects
 				(font
@@
 		)
 		(property "Sim.Pins" "1=K 2=A"
-			(at 77.47 35.56 0)
+			(at 87.63 36.83 0)
 			(effects
 				(font
@@
 	(symbol
 		(lib_id "Device:C_Polarized")
-		(at 88.9 29.21 0)
+		(at 99.06 30.48 0)
 		(unit 1)
 		(exclude_from_sim no)
@@
 		(fields_autoplaced yes)
 		(property "Reference" "C9"
-			(at 92.71 27.0509 0)
+			(at 102.87 28.3209 0)
 			(effects
 				(font
@@
 		)
 		(property "Value" "470uF"
-			(at 92.71 29.5909 0)
+			(at 102.87 30.8609 0)
 			(effects
 				(font
@@
 		)
 		(property "Footprint" ""
-			(at 89.8652 33.02 0)
+			(at 100.0252 34.29 0)
 			(effects
 				(font
@@
 		)
 		(property "Datasheet" "~"
-			(at 88.9 29.21 0)
+			(at 99.06 30.48 0)
 			(effects
 				(font
@@
 		)
 		(property "Description" "Polarized capacitor"
-			(at 88.9 29.21 0)
+			(at 99.06 30.48 0)
 			(effects
 				(font
@@
 	(symbol
 		(lib_id "Device:C")
-		(at 101.6 29.21 0)
+		(at 111.76 30.48 0)
 		(unit 1)
 		(exclude_from_sim no)
@@
 		(fields_autoplaced yes)
 		(property "Reference" "C10"
-			(at 105.41 27.9399 0)
+			(at 115.57 29.2099 0)
 			(effects
 				(font
@@
 		)
 		(property "Value" "100nF"
-			(at 105.41 30.4799 0)
+			(at 115.57 31.7499 0)
 			(effects
 				(font
@@
 		)
 		(property "Footprint" ""
-			(at 102.5652 33.02 0)
+			(at 112.7252 34.29 0)
 			(effects
 				(font
@@
 		)
 		(property "Datasheet" "~"
-			(at 101.6 29.21 0)
+			(at 111.76 30.48 0)
 			(effects
 				(font
@@
 		)
 		(property "Description" "Unpolarized capacitor"
-			(at 101.6 29.21 0)
+			(at 111.76 30.48 0)
 			(effects
 				(font
@@
 	(symbol
 		(lib_id "Device:R")
-		(at 77.47 26.67 0)
+		(at 87.63 27.94 0)
 		(unit 1)
 		(exclude_from_sim no)
@@
 		(fields_autoplaced yes)
 		(property "Reference" "R10"
-			(at 80.01 25.3999 0)
+			(at 90.17 26.6699 0)
 			(effects
 				(font
@@
 		)
 		(property "Value" "330"
-			(at 80.01 27.9399 0)
+			(at 90.17 29.2099 0)
 			(effects
 				(font
@@
 		)
 		(property "Footprint" ""
-			(at 75.692 26.67 90)
+			(at 85.852 27.94 90)
 			(effects
 				(font
@@
 		)
 		(property "Datasheet" "~"
-			(at 77.47 26.67 0)
+			(at 87.63 27.94 0)
 			(effects
 				(font
@@
 		)
 		(property "Description" "Resistor"
-			(at 77.47 26.67 0)
+			(at 87.63 27.94 0)
 			(effects
 				(font
