File: Schematic/MCU_MR/MCU_MR.kicad_sch (KiCad schematic)
At the start: 28 parts, among them J1 USB to TTL CP2102, J2 Power supply terminal, J3 PICKIT3, SW1 SW_Push, SW2 SW_Push, SW3 SW_Push, SW4 SW_Push, U1 PIC16F887-IP, Y1 20MHz

Commit message: Schematic
Connections:
- net LED_G: now also U1.22 (RD3); no longer U1.21 (RD2)
- net LED_R: now also U1.21 (RD2); no longer U1.22 (RD3)
Changed lines of the file:
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@@
 		)
 	)
-	(label "LED_G"
+	(label "LED_R"
 		(at 110.49 83.82 180)
 		(effects
@@
 		)
 	)
-	(label "LED_R"
+	(label "LED_G"
 		(at 110.49 86.36 180)
 		(effects
